File: foras-promineo-revB-em/batteryboard.kicad_sch (KiCad schematic)
At the start: 23 parts, among them J101 KEYSTONE-1042, J102 KEYSTONE-1042, J103 KEYSTONE-1042, J104 KEYSTONE-1042, J105 KEYSTONE-1042, J106 KEYSTONE-1042, Q101 IRF7458, Q102 IRF7458, U101 R5460N233AF

Commit message: final changes before fab
Parts:
- J101: footprint batteryboard-v01b_SLI_card:KEYSTONE-1042_ALT_J1 -> batteryboard:KEYSTONE-1042_ALT_J1
- J102, J104, J106: footprint batteryboard-v01b_SLI_card:KEYSTONE-1042 -> batteryboard:KEYSTONE-1042
- J103: footprint batteryboard-v01b_SLI_card:KEYSTONE-1042_ALT_J5 -> batteryboard:KEYSTONE-1042_ALT_J5
- J105: footprint batteryboard-v01b_SLI_card:KEYSTONE-1042_alt_J4 -> batteryboard:KEYSTONE-1042_alt_J4
- J107: value (none) -> Conn_02x10_Top_Bottom; footprint (none) -> batteryboard:SAMTEC_S2M-110-02-X-D
Other:
- note added: "to add: per parallel line protection? heater?"
- note removed: "to add: per parallel line protection? NTC and heater?"
Changed lines of the file:
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@@
     (effects (font (size 1.905 1.905)) (justify left bottom))
   )
-  (text "to add:\nper parallel line protection?\nNTC and heater?"
-    (at 194.31 34.29 0)
+  (text "to add:\nper parallel line protection?\nheater?" (at 194.31 34.29 0)
     (effects (font (size 1.27 1.27)) (justify left bottom))
   )
@@
     (property "Reference" "J104" (id 0) (at 130.81 63.119 0))
     (property "Value" "KEYSTONE-1042" (id 1) (at 130.81 65.4304 0))
-    (property "Footprint" "batteryboard-v01b_SLI_card:KEYSTONE-1042" (id 2) (at 139.7 67.31 0)
+    (property "Footprint" "batteryboard:KEYSTONE-1042" (id 2) (at 139.7 67.31 0)
       (effects (font (size 1.27 1.27)) (justify left) hide)
     )
@@
     (property "Reference" "J101" (id 0) (at 105.41 63.119 0))
     (property "Value" "KEYSTONE-1042" (id 1) (at 105.41 65.4304 0))
-    (property "Footprint" "batteryboard-v01b_SLI_card:KEYSTONE-1042_ALT_J1" (id 2) (at 114.3 67.31 0)
+    (property "Footprint" "batteryboard:KEYSTONE-1042_ALT_J1" (id 2) (at 114.3 67.31 0)
       (effects (font (size 1.27 1.27)) (justify left) hide)
     )
@@
     (property "Reference" "J102" (id 0) (at 105.41 74.549 0))
     (property "Value" "KEYSTONE-1042" (id 1) (at 105.41 76.8604 0))
-    (property "Footprint" "batteryboard-v01b_SLI_card:KEYSTONE-1042" (id 2) (at 114.3 78.74 0)
+    (property "Footprint" "batteryboard:KEYSTONE-1042" (id 2) (at 114.3 78.74 0)
       (effects (font (size 1.27 1.27)) (justify left) hide)
     )
@@
     (property "Reference" "J105" (id 0) (at 130.81 74.549 0))
     (property "Value" "KEYSTONE-1042" (id 1) (at 130.81 76.8604 0))
-    (property "Footprint" "batteryboard-v01b_SLI_card:KEYSTONE-1042_alt_J4" (id 2) (at 139.7 78.74 0)
+    (property "Footprint" "batteryboard:KEYSTONE-1042_alt_J4" (id 2) (at 139.7 78.74 0)
       (effects (font (size 1.27 1.27)) (justify left) hide)
     )
@@
     (property "Reference" "J103" (id 0) (at 105.41 85.979 0))
     (property "Value" "KEYSTONE-1042" (id 1) (at 105.41 88.2904 0))
-    (property "Footprint" "batteryboard-v01b_SLI_card:KEYSTONE-1042_ALT_J5" (id 2) (at 114.3 90.17 0)
+    (property "Footprint" "batteryboard:KEYSTONE-1042_ALT_J5" (id 2) (at 114.3 90.17 0)
       (effects (font (size 1.27 1.27)) (justify left) hide)
     )
@@
     (property "Reference" "J106" (id 0) (at 130.81 85.979 0))
     (property "Value" "KEYSTONE-1042" (id 1) (at 130.81 88.2904 0))
-    (property "Footprint" "batteryboard-v01b_SLI_card:KEYSTONE-1042" (id 2) (at 139.7 90.17 0)
+    (property "Footprint" "batteryboard:KEYSTONE-1042" (id 2) (at 139.7 90.17 0)
       (effects (font (size 1.27 1.27)) (justify left) hide)
     )
@@
     (in_bom yes) (on_board yes) (fields_autoplaced)
     (property "Reference" "J107" (id 0) (at 209.55 44.45 0))
-    (property "Value" "" (id 1) (at 209.55 46.99 0))
-    (property "Footprint" "" (id 2) (at 208.28 60.96 0)
+    (property "Value" "Conn_02x10_Top_Bottom" (id 1) (at 209.55 46.99 0))
+    (property "Footprint" "batteryboard:SAMTEC_S2M-110-02-X-D" (id 2) (at 208.28 60.96 0)
       (effects (font (size 1.27 1.27)) hide)
     )
@@
     )
     (path "/00000000-0000-0000-0000-00005e17b796"
-      (reference "J101") (unit 1) (value "KEYSTONE-1042") (footprint "batteryboard-v01b_SLI_card:KEYSTONE-1042_ALT_J1")
+      (reference "J101") (unit 1) (value "KEYSTONE-1042") (footprint "batteryboard:KEYSTONE-1042_ALT_J1")
     )
     (path "/00000000-0000-0000-0000-00005e17bc26"
-      (reference "J102") (unit 1) (value "KEYSTONE-1042") (footprint "batteryboard-v01b_SLI_card:KEYSTONE-1042")
+      (reference "J102") (unit 1) (value "KEYSTONE-1042") (footprint "batteryboard:KEYSTONE-1042")
     )
     (path "/00000000-0000-0000-0000-00005e17c580"
-      (reference "J103") (unit 1) (value "KEYSTONE-1042") (footprint "batteryboard-v01b_SLI_card:KEYSTONE-1042_ALT_J5")
+      (reference "J103") (unit 1) (value "KEYSTONE-1042") (footprint "batteryboard:KEYSTONE-1042_ALT_J5")
     )
     (path "/00000000-0000-0000-0000-00005e1793de"
-      (reference "J104") (unit 1) (value "KEYSTONE-1042") (footprint "batteryboard-v01b_SLI_card:KEYSTONE-1042")
+      (reference "J104") (unit 1) (value "KEYSTONE-1042") (footprint "batteryboard:KEYSTONE-1042")
     )
     (path "/00000000-0000-0000-0000-00005e17c1b8"
-      (reference "J105") (unit 1) (value "KEYSTONE-1042") (footprint "batteryboard-v01b_SLI_card:KEYSTONE-1042_alt_J4")
+      (reference "J105") (unit 1) (value "KEYSTONE-1042") (footprint "batteryboard:KEYSTONE-1042_alt_J4")
     )
     (path "/00000000-0000-0000-0000-00005e17c9e0"
-      (reference "J106") (unit 1) (value "KEYSTONE-1042") (footprint "batteryboard-v01b_SLI_card:KEYSTONE-1042")
+      (reference "J106") (unit 1) (value "KEYSTONE-1042") (footprint "batteryboard:KEYSTONE-1042")
     )
     (path "/75e3a46b-a343-4690-928c-fea2c4011b18"
