File: foras-promineo-revB-em/batteryboard.kicad_pcb (KiCad board)
At the start: 2 copper layers, 90.2 x 101.1 mm, 50 parts, among them J101 KEYSTONE-1042, J102 KEYSTONE-1042, J103 KEYSTONE-1042, J104 KEYSTONE-1042, J105 KEYSTONE-1042, J106 KEYSTONE-1042, J107 Conn_02x10_Top_Bottom, P201 Conn_02x60_Top_Bottom, Q101 IRF7458, Q102 IRF7458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

Commit message: FM
Other:
- board text added: "REV: FM"
- board text removed: "revB-em"
Changed lines of the file:
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@@
   (setup
     (stackup
-      (layer "F.SilkS" (type "Top Silk Screen"))
+      (layer "F.SilkS" (type "Top Silk Screen") (color "Black"))
       (layer "F.Paste" (type "Top Solder Paste"))
-      (layer "F.Mask" (type "Top Solder Mask") (color "Blue") (thickness 0.01))
+      (layer "F.Mask" (type "Top Solder Mask") (color "White") (thickness 0.01))
       (layer "F.Cu" (type "copper") (thickness 0.035))
       (layer "dielectric 1" (type "core") (thickness 1.51) (material "FR4") (epsilon_r 4.5) (loss_tangent 0.02))
       (layer "B.Cu" (type "copper") (thickness 0.035))
-      (layer "B.Mask" (type "Bottom Solder Mask") (color "Blue") (thickness 0.01))
+      (layer "B.Mask" (type "Bottom Solder Mask") (color "White") (thickness 0.01))
       (layer "B.Paste" (type "Bottom Solder Paste"))
-      (layer "B.SilkS" (type "Bottom Silk Screen"))
-      (copper_finish "None")
+      (layer "B.SilkS" (type "Bottom Silk Screen") (color "Black"))
+      (copper_finish "ENIG")
       (dielectric_constraints no)
+      (edge_connector bevelled)
     )
     (pad_to_mask_clearance 0.0508)
@@
       (drillshape 0)
       (scaleselection 1)
-      (outputdirectory "gerbers/")
+      (outputdirectory "C:/Users/ckkornowski/Documents/GitHub/batteryboard/FM/")
     )
   )
@@
   (gr_circle (center 87.7189 73.4949) (end 87.7443 73.4187) (layer "F.SilkS") (width 0.4) (fill none))
   (gr_circle (center 81.5975 87.7697) (end 81.6229 87.6935) (layer "F.SilkS") (width 0.4) (fill none))
+  (gr_rect (start 92.559988 102.650011) (end 83.549998 133.130011) (layer "F.SilkS") (width 0.254) (fill none))
   (gr_line (start 109.626402 142.773398) (end 109.626402 142.239998) (layer "Edge.Cuts") (width 0.254))
   (gr_arc (start 110.820202 143.967198) (mid 109.976058 143.617542) (end 109.626402 142.773398) (layer "Edge.Cuts") (width 0.254))
@@
   (gr_line (start 53.238393 142.697198) (end 53.238402 106.933998) (layer "Edge.Cuts") (width 0.254))
   (gr_line (start 69.442154 42.84137) (end 70.222203 42.84137) (layer "Edge.Cuts") (width 0.254))
-  (gr_arc (start 54.356002 143.967198) (mid 53.534176 143.563661) (end 53.238402 142.697198) (layer "Edge.Cuts") (width 0.254))
+  (gr_arc (start 54.356002 143.967198) (mid 53.534175 143.563661) (end 53.238402 142.697198) (layer "Edge.Cuts") (width 0.254))
   (gr_line (start 110.820202 143.967198) (end 142.214602 143.967198) (layer "Edge.Cuts") (width 0.254))
   (gr_line (start 143.408402 142.773398) (end 143.408402 106.933998) (layer "Edge.Cuts") (width 0.254))
@@
     (effects (font (size 1.27 1.016) (thickness 0.254)))
   )
-  (gr_text "revB-em" (at 76.454 142.494) (layer "F.SilkS")
+  (gr_text "REV: FM" (at 72.84 142.64) (layer "F.SilkS")
     (effects (font (size 1.016 1.016) (thickness 0.254)))
   )
