File: revB/batteryboard.kicad_sch (KiCad schematic)
At the start: 23 parts, among them J101 KEYSTONE-1042, J102 KEYSTONE-1042, J103 KEYSTONE-1042, J104 KEYSTONE-1042, J105 KEYSTONE-1042, J106 KEYSTONE-1042, J107 Conn_02x10_Top_Bottom, Q101 IRF7458, Q102 IRF7458, U101 R5460N233AF

Commit message: update project to kicad 7 format
Other:
- note added: "10kΩ, B = 3380 NTC"
- note removed: "10kΩ, B = 3380 NTC for charger IC, but that only allows charging from 0 to 40C, do we want more temp-control on the mainboard side?"
- note removed: "to add: per parallel line protection? heater?"
